Commit message: v2.1

File: berserker_description/urdf/berserker_macro.urdf.xacro (robot description, xacro)
@@ -75,4 +75,5 @@
       <child link="RL_wheel_link"/>
       <axis xyz="0 1 0"/>
+      <mimic joint="FL_wheel_joint" multiplier="1" offset="0"/>
     </joint>
     <link name="RL_wheel_link">
@@ -91,4 +92,5 @@
       <child link="RR_wheel_link"/>
       <axis xyz="0 1 0"/>
+      <mimic joint="FR_wheel_joint" multiplier="1" offset="0"/>
     </joint>
     <link name="RR_wheel_link">
